File: Tester58_PCB/Tester58.kicad_pcb (KiCad board)
At the start: 2 copper layers, 304.4 x 98.8 mm, 119 parts, among them J1 Conn_01x02, SW1 SW_PUSH, SW10 SW_PUSH, SW11 SW_PUSH, SW12 SW_PUSH, SW13 SW_PUSH, SW14 SW_PUSH, SW15 SW_PUSH, SW16 SW_PUSH, SW17 SW_PUSH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

Commit message: fix
Parts:
- SW13, SW14, SW15, SW17, SW18, SW19, SW44, SW45, SW46, SW47: footprint kbd_SW:CherryMX_Choc_Hotswap_1u -> kbd_SW:CherryMX_Hotswap_1u
Routing:
- net Net-(D47-Pad1): track 23.4 -> 6.67 mm

Commit message: fix
Other:
- board text added: "Tester58 v1.0 PCB designed by Fennel"
