File: comfrey77_SWP/comfrey77.kicad_pcb (KiCad board)
At the start: 2 copper layers, 314.4 x 98.8 mm, 74 parts, among them J10 Conn_01x01, J11 Conn_01x01, J12 Conn_01x01, J13 Conn_01x01, J14 Conn_01x01, J15 Conn_01x01, J16 Conn_01x01, J17 Conn_01x01, J2 Conn_01x01, J3 Conn_01x01, J4 Conn_01x01, J5 Conn_01x01, J6 Conn_01x01, J7 Conn_01x01, J8 Conn_01x01, J9 Conn_01x01, SW1 SW_PUSH, SW10 SW_PUSH, SW11 SW_PUSH, SW12 SW_PUSH, SW13 SW_PUSH, SW14 SW_PUSH, SW15 SW_PUSH, SW16 SW_PUSH, SW17 SW_PUSH, SW18 SW_PUSH, SW19 SW_PUSH, SW2 SW_PUSH, SW20 SW_PUSH, SW21 SW_PUSH, SW22 SW_PUSH, SW23 SW_PUSH, SW24 KEY_SWITCH, SW25 SW_PUSH, SW26 SW_PUSH, SW27 SW_PUSH, SW28 SW_PUSH, SW29 SW_PUSH, SW3 SW_PUSH, SW30 SW_PUSH, SW31 SW_PUSH, SW32 SW_PUSH, SW33 SW_PUSH, SW34 SW_PUSH, SW35 SW_PUSH, SW36 SW_PUSH, SW37 SW_PUSH, SW38 KEY_SWITCH, SW39 SW_PUSH, SW4 KEY_SWITCH, SW40 SW_PUSH, SW41 SW_PUSH, SW42 SW_PUSH, SW43 SW_PUSH, SW44 SW_PUSH, SW45 SW_PUSH, SW46 SW_PUSH, SW47 SW_PUSH, SW48 SW_PUSH, SW49 SW_PUSH, SW5 SW_PUSH, SW50 SW_PUSH, SW51 SW_PUSH, SW52 SW_PUSH, SW53 SW_PUSH, SW54 SW_PUSH, SW55 SW_PUSH, SW56 SW_PUSH, SW57 SW_PUSH, SW58 KEY_SWITCH, SW6 SW_PUSH, SW7 SW_PUSH, SW8 SW_PUSH, SW9 SW_PUSH

Commit message: add LOGO
Parts:
- removed SW10, SW14, SW15, SW18, SW19, SW2, SW20, SW23, SW29, SW3, SW30, SW33, SW34, SW35, SW39, SW40, SW43, SW44, SW45, SW48, SW49, SW50, SW53, SW54, SW8: SW_PUSH, kbd_SW_Hole:SW_Hole_1u
- removed the SW11 at (70.5, 72.7)
- removed the SW12 at (79.6, 94.8)
- removed the SW16 at (100.4, 97.8)
- removed the SW22 at (128.7, 62.9)
- removed SW24, SW38, SW4: KEY_SWITCH, kbd_SW_Hole:SW_Hole_1.5u
- removed the SW26 at (152.4, 47.6)
- removed the SW27 at (152.4, 66.7)
- removed the SW32 at (190.5, 47.6)
- removed the SW36 at (214.2, 62.8)
- removed the SW37 at (215.8, 81.8)
- removed the SW41 at (234.5, 75.9)
- removed the SW42 at (221.5, 102.4)
- removed the SW46 at (242.5, 97.8)
- removed the SW57 at (310.7, 73.5)
- removed the SW58 at (307.6, 92.9)
- removed the SW6 at (53.0, 54.1)
- removed the SW7 at (51.3, 73.1)
- added SW1: SW_PUSH, kbd_SW_Hole:SW_Hole_1u, F.Cu at (28.6, 85.7)
- added SW1: SW_PUSH, kbd_SW_Hole:SW_Hole_1u, F.Cu at (28.6, 28.6)
- added SW11: SW_PUSH, kbd_SW_Hole:SW_Hole_1u, F.Cu at (66.7, 85.7)
- added SW11: SW_PUSH, kbd_SW_Hole:SW_Hole_1u, F.Cu at (66.7, 28.6)
- added SW12: SW_PUSH, kbd_SW_Hole:SW_Hole_1u, F.Cu at (57.1, 104.8)
- added SW12: SW_PUSH, kbd_SW_Hole:SW_Hole_1u, F.Cu at (57.1, 66.7)
- added SW16: SW_PUSH, kbd_SW_Hole:SW_Hole_1u, F.Cu at (85.7, 85.7)
- added SW16: SW_PUSH, kbd_SW_Hole:SW_Hole_1u, F.Cu at (85.7, 28.6)
- added SW17: SW_PUSH, kbd_SW_Hole:SW_Hole_1u, F.Cu at (76.2, 104.8)
- added SW17: SW_PUSH, kbd_SW_Hole:SW_Hole_1u, F.Cu at (76.2, 66.7)
- added SW21: SW_PUSH, kbd_SW_Hole:SW_Hole_1u, F.Cu at (104.8, 85.7)
- added SW21: SW_PUSH, kbd_SW_Hole:SW_Hole_1u, F.Cu at (104.8, 28.6)
- added SW22: SW_PUSH, kbd_SW_Hole:SW_Hole_1u, F.Cu at (95.2, 104.8)
- added SW22: SW_PUSH, kbd_SW_Hole:SW_Hole_1u, F.Cu at (95.2, 66.7)
- added SW26: SW_PUSH, kbd_SW_Hole:SW_Hole_1u, F.Cu at (123.8, 85.7)
- added SW26: SW_PUSH, kbd_SW_Hole:SW_Hole_1u, F.Cu at (123.8, 28.6)
- added SW27: SW_PUSH, kbd_SW_Hole:SW_Hole_1u, F.Cu at (114.3, 104.8)
- added SW27: SW_PUSH, kbd_SW_Hole:SW_Hole_1u, F.Cu at (114.3, 66.7)
- added SW31: SW_PUSH, kbd_SW_Hole:SW_Hole_1u, F.Cu at (142.9, 85.7)
- added SW31: SW_PUSH, kbd_SW_Hole:SW_Hole_1u, F.Cu at (142.9, 28.6)
- added SW32: SW_PUSH, kbd_SW_Hole:SW_Hole_1u, F.Cu at (133.3, 104.8)
- added SW32: SW_PUSH, kbd_SW_Hole:SW_Hole_1u, F.Cu at (133.3, 66.7)
- added SW36: SW_PUSH, kbd_SW_Hole:SW_Hole_1u, F.Cu at (161.9, 85.7)
- added SW36: SW_PUSH, kbd_SW_Hole:SW_Hole_1u, F.Cu at (161.9, 28.6)
- added SW37: SW_PUSH, kbd_SW_Hole:SW_Hole_1u, F.Cu at (152.4, 104.8)
- added SW37: SW_PUSH, kbd_SW_Hole:SW_Hole_1u, F.Cu at (152.4, 66.7)
- added SW41: SW_PUSH, kbd_SW_Hole:SW_Hole_1u, F.Cu at (181.0, 85.7)
- added SW41: SW_PUSH, kbd_SW_Hole:SW_Hole_1u, F.Cu at (181.0, 28.6)
- added SW42: SW_PUSH, kbd_SW_Hole:SW_Hole_1u, F.Cu at (171.4, 104.8)
- added SW42: SW_PUSH, kbd_SW_Hole:SW_Hole_1u, F.Cu at (171.4, 66.7)
- added SW46: SW_PUSH, kbd_SW_Hole:SW_Hole_1u, F.Cu at (200.0, 85.7)
- added SW46: SW_PUSH, kbd_SW_Hole:SW_Hole_1u, F.Cu at (200.0, 28.6)
- added SW47: SW_PUSH, kbd_SW_Hole:SW_Hole_1u, F.Cu at (190.5, 104.8)
- added SW47: SW_PUSH, kbd_SW_Hole:SW_Hole_1u, F.Cu at (190.5, 66.7)
- added SW51: SW_PUSH, kbd_SW_Hole:SW_Hole_1u, F.Cu at (219.1, 85.7)
- added SW51: SW_PUSH, kbd_SW_Hole:SW_Hole_1u, F.Cu at (219.1, 28.6)
- added SW52: SW_PUSH, kbd_SW_Hole:SW_Hole_1u, F.Cu at (209.6, 104.8)
- added SW52: SW_PUSH, kbd_SW_Hole:SW_Hole_1u, F.Cu at (209.6, 66.7)
- added SW56: SW_PUSH, kbd_SW_Hole:SW_Hole_1u, F.Cu at (238.1, 85.7)
- added SW56: SW_PUSH, kbd_SW_Hole:SW_Hole_1u, F.Cu at (238.1, 28.6)
- added SW57: SW_PUSH, kbd_SW_Hole:SW_Hole_1u, F.Cu at (228.6, 104.8)
- added SW57: SW_PUSH, kbd_SW_Hole:SW_Hole_1u, F.Cu at (228.6, 66.7)
- added SW58: SW_PUSH, kbd_SW_Hole:SW_Hole_1u, F.Cu at (285.8, 104.8)
- added SW58: SW_PUSH, kbd_SW_Hole:SW_Hole_1u, F.Cu at (285.8, 66.7)
- added SW59: SW_PUSH, kbd_SW_Hole:SW_Hole_1u, F.Cu at (257.2, 85.7)
- added SW59: SW_PUSH, kbd_SW_Hole:SW_Hole_1u, F.Cu at (257.2, 28.6)
- added SW6: SW_PUSH, kbd_SW_Hole:SW_Hole_1u, F.Cu at (47.6, 85.7)
- added SW6: SW_PUSH, kbd_SW_Hole:SW_Hole_1u, F.Cu at (47.6, 28.6)
- added SW60: SW_PUSH, kbd_SW_Hole:SW_Hole_1u, F.Cu at (247.7, 104.8)
- added SW60: SW_PUSH, kbd_SW_Hole:SW_Hole_1u, F.Cu at (247.7, 66.7)
- added SW61: SW_PUSH, kbd_SW_Hole:SW_Hole_1u, F.Cu at (266.7, 104.8)
- added SW61: SW_PUSH, kbd_SW_Hole:SW_Hole_1u, F.Cu at (266.7, 66.7)
- added SW64: SW_PUSH, kbd_SW_Hole:SW_Hole_1u, F.Cu at (276.2, 85.7)
- added SW64: SW_PUSH, kbd_SW_Hole:SW_Hole_1u, F.Cu at (276.2, 28.6)
- added SW65: SW_PUSH, kbd_SW_Hole:SW_Hole_1u, F.Cu at (295.3, 85.7)
- added SW65: SW_PUSH, kbd_SW_Hole:SW_Hole_1u, F.Cu at (295.3, 28.6)
- added SW69: SW_PUSH, kbd_SW_Hole:SW_Hole_1u, F.Cu at (314.3, 85.7)
- added SW69: SW_PUSH, kbd_SW_Hole:SW_Hole_1u, F.Cu at (314.3, 28.6)
- added SW7: SW_PUSH, kbd_SW_Hole:SW_Hole_1u, F.Cu at (38.1, 104.8)
- added SW7: SW_PUSH, kbd_SW_Hole:SW_Hole_1u, F.Cu at (38.1, 66.7)
- added SW70: SW_PUSH, kbd_SW_Hole:SW_Hole_1u, F.Cu at (304.8, 104.8)
- added SW70: SW_PUSH, kbd_SW_Hole:SW_Hole_1u, F.Cu at (304.8, 66.7)
- added SW70: SW_PUSH, kbd_SW_Hole:SW_Hole_1u, F.Cu at (304.8, 47.6)
- moved SW60 61.0 mm to (247.7, 47.6), turned to 0 degrees
- moved SW57 60.9 mm to (228.6, 47.6), turned to 0 degrees
- moved SW52 60.9 mm to (209.6, 47.6), turned to 0 degrees
- moved SW61 42.9 mm to (266.7, 47.6), turned to 0 degrees
- moved SW37 19.1 mm to (152.4, 47.6)
- moved SW42 19.1 mm to (171.4, 47.6)
- moved SW47 19.1 mm to (190.5, 47.6)
- moved SW22 13.5 mm to (95.2, 47.6), turned to 0 degrees
- moved SW17 13.1 mm to (76.2, 47.6), turned to 0 degrees
- moved SW12 12.8 mm to (57.1, 47.6), turned to 0 degrees
- moved SW7 12.3 mm to (38.1, 47.6), turned to 0 degrees
- moved SW27 9.87 mm to (114.3, 47.6), turned to 0 degrees
- moved SW58 7.66 mm to (285.8, 47.6), turned to 0 degrees
- moved SW32 4.74 mm to (133.3, 47.6), turned to 0 degrees
- renumbered SW5 to SW12, SW9 to SW17, SW13 to SW22, SW17 to SW27, SW21 to SW32, SW25 to SW37, SW28 to SW42, SW31 to SW47, SW47 to SW52, SW51 to SW57, SW52 to SW58, SW55 to SW60, SW56 to SW61, SW1 to SW7
